Commit message: Add necessary file changes for Gazebo launch

File: niryo_one_description/urdf/v1/niryo_one.urdf.xacro (robot description, xacro)
@@ -1,18 +1,3 @@
 <?xml version="1.0"?>
-<!--
-    niryo_one.urdf.xacro
-    Copyright (C) 2017 Niryo
-    All rights reserved.
-    This program is free software: you can redistribute it and/or modify
-    it under the terms of the GNU General Public License as published by
-    the Free Software Foundation, either version 3 of the License, or
-    (at your option) any later version.
-    This program is distributed in the hope that it will be useful,
-    but WITHOUT ANY WARRANTY; without even the implied warranty of
-    MERCHANTABILITY or FITNESS FOR A PARTICULAR PURPOSE.  See the
-    GNU General Public License for more details.
-    You should have received a copy of the GNU General Public License
-    along with this program.  If not, see <http://www.gnu.org/licenses/>.
--->
 <robot xmlns:xacro="http://www.ros.org/wiki/xacro" name="niryo_one">
 	<!-- Properties -->
@@ -40,6 +25,14 @@
     <xacro:property name="limit_low_hand_rotation" value="-2.57" />
     <xacro:property name="limit_up_hand_rotation" value="2.57" />
-	<!-- Links -->
+<!-- ros_control plugin -->
+  <gazebo>
+    <plugin name="gazebo_ros_control" filename="libgazebo_ros_control.so">
+      <robotNamespace>/niryo_one</robotNamespace>
+      <robotSimType>gazebo_ros_control/DefaultRobotHWSim</robotSimType>
+    </plugin>
+  </gazebo>
+<!-- Links -->
     <link name="ground_link"/>
+<!-- ................................................................... -->
     <link name="base_link">
 		<visual>
@@ -52,4 +45,9 @@
 			</material>
         </visual>
+    <inertial>
+      <origin rpy="0 0 0" xyz="0.000000 0.000000 0.000000"/>
+      <mass value="3533.6455"/>
+      <inertia ixx="184.9155" ixy="-0.0354" ixz="-15.4188" iyy="166.2671" iyz="0.3292" izz="80.2239"/>
+    </inertial>
         <collision>
 			<origin xyz="0 0 0" rpy="0 0 0" />
@@ -59,4 +57,5 @@
         </collision>
 	</link>
+<!-- ................................................................... -->
     <link name="shoulder_link">
 		<visual>
@@ -69,4 +68,9 @@
 			</material>
 		</visual>
+    <inertial>
+      <origin rpy="0 0 0" xyz="0.000000 0.000000 0.000000"/>
+      <mass value="0.035336455"/>
+      <inertia ixx="0.001849155" ixy="-0.000000354" ixz="-0.000154188" iyy="0.001662671" iyz="0.000003292" izz="0.000802239"/>
+    </inertial>
         <collision>
 			<origin xyz="0 0 0" rpy="0 0 0" />
@@ -76,4 +80,5 @@
         </collision>
 	</link>
+<!-- ................................................................... -->
     <link name="arm_link">
 		<visual>
@@ -86,4 +91,9 @@
 			</material>
 		</visual>
+    <inertial>
+      <origin rpy="0 0 0" xyz="0.000000 0.000000 0.000000"/>
+      <mass value="0.035336455"/>
+      <inertia ixx="0.001849155" ixy="-0.000000354" ixz="-0.000154188" iyy="0.001662671" iyz="0.000003292" izz="0.000802239"/>
+    </inertial>
         <collision>
 			<origin xyz="0 0 0" rpy="0 0 0" />
@@ -93,4 +103,5 @@
         </collision>
 	</link>
+<!-- ................................................................... -->
     <link name="elbow_link">
 		<visual>
@@ -104,4 +115,9 @@
 			</material>
 		</visual>
+    <inertial>
+      <origin rpy="0 0 0" xyz="0.000000 0.000000 0.000000"/>
+      <mass value="0.035336455"/>
+      <inertia ixx="0.001849155" ixy="-0.000000354" ixz="-0.000154188" iyy="0.001662671" iyz="0.000003292" izz="0.000802239"/>
+    </inertial>
         <collision>
 			<origin xyz="0 0 0" rpy="0 0 0" />
@@ -111,4 +127,5 @@
         </collision>
 	</link>
+<!-- ................................................................... -->
     <link name="forearm_link">
 		<visual>
@@ -121,4 +138,9 @@
 			</material>
 		</visual>
+    <inertial>
+      <origin rpy="0 0 0" xyz="0.000000 0.000000 0.000000"/>
+      <mass value="0.035336455"/>
+      <inertia ixx="0.001849155" ixy="-0.000000354" ixz="-0.000154188" iyy="0.001662671" iyz="0.000003292" izz="0.000802239"/>
+    </inertial>
         <collision>
 			<origin xyz="0 0 0" rpy="0 0 0" />
@@ -128,4 +150,5 @@
         </collision>
 	</link>
+<!-- ................................................................... -->
     <link name="wrist_link">
 		<visual>
@@ -138,4 +161,9 @@
 			</material>
 		</visual>
+    <inertial>
+      <origin rpy="0 0 0" xyz="0.000000 0.000000 0.000000"/>
+      <mass value="0.035336455"/>
+      <inertia ixx="0.001849155" ixy="-0.000000354" ixz="-0.000154188" iyy="0.001662671" iyz="0.000003292" izz="0.000802239"/>
+    </inertial>
         <collision>
 			<origin xyz="0 0 0" rpy="0 0 0" />
@@ -145,4 +173,5 @@
         </collision>
 	</link>
+<!-- ................................................................... -->
     <link name="hand_link">
 		<visual>
@@ -155,4 +184,9 @@
 			</material>
 		</visual>
+    <inertial>
+      <origin rpy="0 0 0" xyz="0.000000 0.000000 0.000000"/>
+      <mass value="0.035336455"/>
+      <inertia ixx="0.001849155" ixy="-0.000000354" ixz="-0.000154188" iyy="0.001662671" iyz="0.000003292" izz="0.000802239"/>
+    </inertial>
         <collision>
 			<origin xyz="0 0 0" rpy="0 0 0" />
@@ -162,7 +196,8 @@
         </collision>
 	</link>
+<!-- ................................................................... -->
     <link name="tool_link">
 	</link>
-	<!--Joints -->
+<!--Joints -->
     <joint name="ground_joint" type="fixed">
         <parent link="ground_link" />
@@ -170,4 +205,5 @@
         <origin xyz="0 0 0" rpy="0 0 0" />
     </joint>
+<!-- ................................................................... -->
 	<joint name="joint_1" type="revolute">
         <parent link="base_link" />
@@ -177,4 +213,5 @@
 		<limit effort="1" velocity="1.0" lower="${limit_low_shoulder_rotation}" upper="${limit_up_shoulder_rotation}" />
 	</joint>
+<!-- ................................................................... -->
 	<joint name="joint_2" type="revolute">
         <parent link="shoulder_link" />
@@ -184,4 +221,5 @@
 		<axis xyz="0 0 1" />
 	</joint>
+<!-- ................................................................... -->
 	<joint name="joint_3" type="revolute">
         <parent link="arm_link" />
@@ -191,4 +229,5 @@
 		<axis xyz="0 0 1" />
 	</joint>
+<!-- ................................................................... -->
 	<joint name="joint_4" type="revolute">
         <parent link="elbow_link" />
@@ -198,4 +237,5 @@
 		<axis xyz="0 0 1" />
 	</joint>
+<!-- ................................................................... -->
 	<joint name="joint_5" type="revolute">
         <parent link="forearm_link" />
@@ -205,4 +245,5 @@
 		<axis xyz="0 0 1" />
 	</joint>
+<!-- ................................................................... -->
 	<joint name="joint_6" type="revolute">
         <parent link="wrist_link" />
@@ -212,4 +253,5 @@
 		<axis xyz="0 0 1" />
 	</joint>
+<!-- ................................................................... -->
 	<joint name="hand_tool_joint" type="fixed">
         <parent link="hand_link" />
@@ -217,3 +259,69 @@
         <origin xyz="0 0 ${distance_hand_tool}" rpy="${-PI/2} ${-PI/2} 0" />
 	</joint>
+<!-- Transmission -->
+  <transmission name="tran1">
+    <type>transmission_interface/SimpleTransmission</type>
+    <joint name="joint_1">
+      <hardwareInterface>hardware_interface/PositionJointInterface</hardwareInterface>
+    </joint>
+    <actuator name="motor1">
+      <hardwareInterface>hardware_interface/PositionJointInterface</hardwareInterface>
+      <mechanicalReduction>10000000000000</mechanicalReduction>
+    </actuator>
+  </transmission>
+<!-- ................................................................... -->
+  <transmission name="tran2">
+    <type>transmission_interface/SimpleTransmission</type>
+    <joint name="joint_2">
+      <hardwareInterface>hardware_interface/PositionJointInterface</hardwareInterface>
+    </joint>
+    <actuator name="motor2">
+      <hardwareInterface>hardware_interface/PositionJointInterface</hardwareInterface>
+      <mechanicalReduction>1000000000000000000000000000</mechanicalReduction>
+    </actuator>
+  </transmission>
+<!-- ................................................................... -->
+  <transmission name="tran3">
+    <type>transmission_interface/SimpleTransmission</type>
+    <joint name="joint_3">
+      <hardwareInterface>hardware_interface/PositionJointInterface</hardwareInterface>
+    </joint>
+    <actuator name="motor3">
+      <hardwareInterface>hardware_interface/PositionJointInterface</hardwareInterface>
+      <mechanicalReduction>10000000000000</mechanicalReduction>
+    </actuator>
+  </transmission>
+<!-- ................................................................... -->
+  <transmission name="tran4">
+    <type>transmission_interface/SimpleTransmission</type>
+    <joint name="joint_4">
+      <hardwareInterface>hardware_interface/PositionJointInterface</hardwareInterface>
+    </joint>
+    <actuator name="motor4">
+      <hardwareInterface>hardware_interface/PositionJointInterface</hardwareInterface>
+      <mechanicalReduction>10000000000000</mechanicalReduction>
+    </actuator>
+  </transmission>
+<!-- ................................................................... -->
+  <transmission name="tran5">
+    <type>transmission_interface/SimpleTransmission</type>
+    <joint name="joint_5">
+      <hardwareInterface>hardware_interface/PositionJointInterface</hardwareInterface>
+    </joint>
+    <actuator name="motor5">
+      <hardwareInterface>hardware_interface/PositionJointInterface</hardwareInterface>
+      <mechanicalReduction>10000000000000</mechanicalReduction>
+    </actuator>
+  </transmission>
+<!-- ................................................................... -->
+  <transmission name="tran6">
+    <type>transmission_interface/SimpleTransmission</type>
+    <joint name="joint_6">
+      <hardwareInterface>hardware_interface/PositionJointInterface</hardwareInterface>
+    </joint>
+    <actuator name="motor6">
+      <hardwareInterface>hardware_interface/PositionJointInterface</hardwareInterface>
+      <mechanicalReduction>10000000000000</mechanicalReduction>
+    </actuator>
+  </transmission>
 </robot>
